Commit message: repair the laser X position

File: src/robot_description/urdf/robot_base.urdf (robot description, URDF)
Before this commit: robot robot, 6 links, 5 joints
Joints:
- joint laser_joint: origin xyz=0.15 0 0.05 -> xyz=0.015 0 0.05

Commit message: repair the urdf caster_joint type be the fixed

File: src/robot_description/urdf/robot_base.urdf (robot description, URDF)
Before this commit: robot robot, 6 links, 5 joints
Joints:
- joint front_caster_joint: type continuous -> fixed

Commit message: cartographer build map test success , robot_cartographer.launch.py launch all files except  rviz2

File: src/robot_description/urdf/robot_base.urdf (robot description, URDF)
Before this commit: robot robot, 7 links, 6 joints
Joints:
- joint laser_joint: origin xyz=0.015 0 0.05 -> xyz=0.015 0 0.05 rpy=0 0 3.1415926
